File: Blade.kicad_sch (KiCad schematic)
At the start: 64 parts, among them J1 Connector, USB-TYPE-C-16P, J2 Connector, USB-TYPE-C-16P, J3 Conn_ARM_JTAG_SWD_10, Q1 SI2301CDS-T1-GE3, Q2 BSS138, Q3 BSS138, Q4 IRLML6344, Q5 MMBT3904LT1G, Q6 MMBT3904LT1G, SW1 BSI-10, U1 ESP32-S3-WROOM-1-N16, U2 CH340G, U3 AMS1117, U4 AP2112K-1.8, U5 TXS0108EPW, U6 W25Q128, U7 AT24C256C, U8 INA219AIDR, U9 TSOP382xx

Commit message: Add redirection page for import guide
Parts:
- removed SJ1, SJ2: SolderJumper_2_Open, Jumper:SolderJumper-2_P1.3mm_Open_RoundedPad1.0x1.5mm, symbol Jumper:SolderJumper_2_Open
- removed U2: CH340G, PCM_JLCPCB:SOIC-16_3.9x9.9mm_P1.27mm, symbol PCM_JLCPCB-Extended:USB-Serial, CH340G
- removed U8: INA219AIDR, Package_SO:SOIC-8_3.9x4.9mm_P1.27mm, symbol Sensor_Energy:INA219AxDCN
- added C18, C7: 10uF, PCM_JLCPCB:C_0603, symbol PCM_JLCPCB-Capacitors:0603,10uF
- added C19, C20, C22, C23, C24, C25, C26, C27, C28, C29, C30, C31, C8: 100nF, PCM_JLCPCB:C_0402, symbol PCM_JLCPCB-Capacitors:0402,100nF
- added C9: 1uF, PCM_JLCPCB:C_0603, symbol PCM_JLCPCB-Capacitors:0603,1uF
- added D3: White, PCM_JLCPCB:D_0603, symbol PCM_JLCPCB-Diodes:LED,0603,White
- added D4: Green, PCM_JLCPCB:D_0805, symbol PCM_JLCPCB-Diodes:LED,0805,Green
- added J10: 2x10 Conn, Connector_PinHeader_2.54mm:PinHeader_2x10_P2.54mm_Vertical, symbol Connector_Generic:Conn_02x10_Odd_Even
- added J11: 1x2 Conn, Connector_PinHeader_2.54mm:PinHeader_1x02_P2.54mm_Vertical, symbol Connector:Conn_01x02_Pin
- added J12, J13: 1x3 Conn, Connector_PinHeader_2.54mm:PinHeader_1x03_P2.54mm_Vertical, symbol Connector:Conn_01x03_Pin
- added J4: 1x8 Conn, Connector_PinHeader_2.54mm:PinHeader_1x08_P2.54mm_Vertical, symbol Connector:Conn_01x08_Pin
- added J5: 1x6 Conn, Connector_PinHeader_2.54mm:PinHeader_1x06_P2.54mm_Vertical, symbol Connector:Conn_01x06_Pin
- added J6, J9: 1x4 Conn, Connector_PinHeader_2.54mm:PinHeader_1x04_P2.54mm_Vertical, symbol Connector:Conn_01x04_Pin
- added J7: 5025700893, Connector_Card:MOLEX_5025700893, symbol Connector:5025700893
- added J8: SOIC-8 Conn, Connector_PinHeader_2.54mm:PinHeader_2x04_P2.54mm_Vertical_Counter_Clockwise, symbol Connector_Generic:Conn_02x04_Counter_Clockwise
- added LED2: Red, PCM_JLCPCB:D_0603, symbol PCM_JLCPCB-Diodes:LED,0603,Red
- added LED4, LED5, LED6, LED7, LED8, LED9: WS2812B, LED_SMD:LED_WS2812B_PLCC4_5.0x5.0mm_P3.2mm, symbol LED:WS2812B
- added R14, R16, R26, R27, R28, R29, R32, R6, R7: 10kΩ, PCM_JLCPCB:R_0805, symbol PCM_JLCPCB-Resistors:0805,10kΩ
- added R19, R30, R5: 1kΩ, PCM_JLCPCB:R_0805, symbol PCM_JLCPCB-Resistors:0805,1kΩ
- added R25: 330Ω, PCM_JLCPCB:R_0805, symbol PCM_JLCPCB-Resistors:0805,330Ω
- added SJ1, SJ2: SolderJumper_2_Bridged, Jumper:SolderJumper-2_P1.3mm_Bridged_RoundedPad1.0x1.5mm, symbol Jumper:SolderJumper_2_Bridged
- added SW2: BOOT, PCM_JLCPCB:SW_TS-1088-AR02016, symbol PCM_JLCPCB-Connectors_Buttons:Tactile Button, 160gf, 12V, 50mA, 4.0mm
- added SW3: EN, PCM_JLCPCB:SW_TS-1088-AR02016, symbol PCM_JLCPCB-Connectors_Buttons:Tactile Button, 160gf, 12V, 50mA, 4.0mm
- added SW4: UP, PCM_JLCPCB:SW_TS-1088-AR02016, symbol PCM_JLCPCB-Connectors_Buttons:Tactile Button, 160gf, 12V, 50mA, 4.0mm
- added SW5: DOWN, PCM_JLCPCB:SW_TS-1088-AR02016, symbol PCM_JLCPCB-Connectors_Buttons:Tactile Button, 160gf, 12V, 50mA, 4.0mm
- added SW6: SEL, PCM_JLCPCB:SW_TS-1088-AR02016, symbol PCM_JLCPCB-Connectors_Buttons:Tactile Button, 160gf, 12V, 50mA, 4.0mm
- added SW7: BACK, PCM_JLCPCB:SW_TS-1088-AR02016, symbol PCM_JLCPCB-Connectors_Buttons:Tactile Button, 160gf, 12V, 50mA, 4.0mm
- added U2: CH340C, Package_SO:SOIC-16_3.9x9.9mm_P1.27mm, symbol Interface_USB:CH340C
- added U8: INA219AxD, Package_SO:SOIC-8_3.9x4.9mm_P1.27mm, symbol Sensor_Energy:INA219AxD
- BZ1: LCSC (none) -> C3812310
- D1: LCSC (none) -> C55528
- J3: footprint Connector_PinHeader_1.27mm:PinHeader_2x05_P1.27mm_Vertical -> Connector:Tag-Connect_TC2050-IDC-FP_2x05_P1.27mm_Vertical
- renumbered C7 to C888, R1 to R10, R2 to R24, R3 to R31, R6 to R888, R_SHUNT to R_SHUNT1
Connections:
- net +1V8: now also J10.17 (Pin_17), J12.1 (Pin_1), J13.1 (Pin_1)
- net +3.3V: now also U1.2 (3V3), C18.1, C19.1, C7.1, C8.1, J10.1 (Pin_1), J12.3 (Pin_3), J13.3 (Pin_3), J7.4 (VDD), J9.2 (Pin_2), R14.1, R16.2, R19.2, R26.1, R27.1, R28.1, R29.1, R32.1, R5.1, R6.1, R7.1, SJ1.2 (B), SJ2.2 (B), U2.16 (VCC), U2.4 (V3), U8.5 (VS); no longer C21.1
- net BTN_BOOT: now also U1.27 (IO0), J10.16 (Pin_16), R7.2, SW2.1 (A)
- net BUZZER: now also U1.39 (IO1)
- net CH340_DTR: now also U2.13 (~{DTR})
- net ESP_EN: now also U1.3 (EN), C9.1, J10.15 (Pin_15), R6.2, SW3.1 (A)
- net FLASH_HOLD: now also R14.2; no longer C15.1, U6.8 (VCC)
- net GLITCH_OUT: now also J11.1 (Pin_1)
- net GLITCH_TRIG: now also R17.1, U1.4 (IO4); no longer SW1.3 (A)
- net GND: now also C18.2, C19.2, C20.2, C22.2, C23.2, C24.2, C25.2, C26.2, C27.2, C28.2, C29.2, C30.2, C31.2, C7.2, C8.2, C9.2, D3.2, D4.2, J10.19 (Pin_19), J10.20 (Pin_20), J11.2 (Pin_2), J4.2 (Pin_2), J5.1 (Pin_1), J6.4 (Pin_4), J7.10 (DET_SW), J7.6 (VSS), J8.4 (Pin_4), J9.1 (Pin_1), LED4.3 (VSS), LED5.3 (VSS), LED6.3 (VSS), LED7.3 (VSS), LED8.3 (VSS), LED9.3 (VSS), SW2.2 (B), SW3.2 (B), SW4.2 (B), SW5.2 (B), SW6.2 (B), SW7.2 (B), U2.1 (GND), U8.1 (A1), U8.2 (A0), U8.6 (GND)
- net HI2C_SCL: now also J6.2 (Pin_2)
- net HI2C_SDA: now also J6.3 (Pin_3)
- net HLS_SPARE1: now also J10.8 (Pin_8)
- net HLS_SPARE2: now also J10.10 (Pin_10)
- net HSPI_CS: now also J4.7 (Pin_7), J8.1 (Pin_1)
- net HSPI_MISO: now also J4.5 (Pin_5), J8.2 (Pin_2)
- net HSPI_MOSI: now also J4.3 (Pin_3), J8.5 (Pin_5)
- net HSPI_SCLK: now also J4.4 (Pin_4), J8.6 (Pin_6)
- net HUART_RX: now also J5.5 (Pin_5)
- net HUART_TX: now also J5.4 (Pin_4)
- net I2C_SCL: now also U1.17 (IO9), J10.12 (Pin_12), J9.4 (Pin_4), U8.4 (SCL)
- net I2C_SDA: now also U1.12 (IO8), J10.11 (Pin_11), J9.3 (Pin_3), U8.3 (SDA)
- net IR_RX: now also U1.23 (IO21)
- net IR_TX: now also U1.24 (IO47)
- net IR_VCC: now also C21.1, C20.1
- net JTAG_TCK: now also U1.32 (IO39)
- net JTAG_TDI: now also U1.34 (IO41)
- net JTAG_TDO: now also U1.33 (IO40)
- net JTAG_TMS: now also U1.35 (IO42)
- net LS_SPARE1: now also J10.7 (Pin_7)
- net LS_SPARE2: now also J10.9 (Pin_9)
- net SHIELD1: no longer C888.1, J2.S1 (SHIELD), R888.1
- net SPI_CS_FLASH: now also U1.22 (IO14)
- net SPI_CS_TGT: now also U1.18 (IO10)
- net SPI_MISO: now also U1.21 (IO13), J7.7 (DAT0)
- net SPI_MOSI: now also U1.19 (IO11), J7.3 (CMD)
- net SPI_SCLK: now also U1.20 (IO12), J7.5 (CLK)
- net TGT_PWR_EN: now also U1.5 (IO5)
- net UART0_RXD: now also U1.36 (RXD0), J10.14 (Pin_14), U2.2 (TXD)
- net UART0_TXD: now also U1.37 (TXD0), J10.13 (Pin_13), U2.3 (RXD)
- net UART1_RXD: now also U1.11 (IO18)
- net UART1_TXD: now also U1.10 (IO17)
- net USB1_DN: now also U2.6 (UD-)
- net USB1_DP: now also U2.5 (UD+)
- net USB_DN: now also U1.13 (IO19)
- net USB_DP: now also U1.14 (IO20)
- net VCC_5V: now also C22.1, C23.1, C24.1, C25.1, C26.1, C27.1, J10.2 (Pin_2), LED4.1 (VDD), LED5.1 (VDD), LED6.1 (VDD), LED7.1 (VDD), LED8.1 (VDD), LED9.1 (VDD)
- net VCC_TGT: now also J10.18 (Pin_18), J4.1 (Pin_1), J4.6 (Pin_6), J4.8 (Pin_8), J5.3 (Pin_3), J6.1 (Pin_1), J8.3 (Pin_3), J8.7 (Pin_7), J8.8 (Pin_8)
- net VCC_TGT_IN: now also J12.2 (Pin_2), U8.8 (IN+)
- net VCC_TGT_IO: now also J13.2 (Pin_2)
- net VCC_TGT_OUT: now also U8.7 (IN-)
- net at C16.1, U7.8 (VCC): now also SJ2.1 (A)
- net CH340_RTS: now reaches C12.1
- net CH340_RTS: now also U2.14 (~{RTS})
- net BTN_SEL: now reaches U1.15 (IO3)
- net BTN_SEL: now also C30.1, R28.2, SW6.1 (A)
- net BTN_DOWN: now reaches U1.16 (IO46)
- net BTN_DOWN: now also C29.1, R27.2, SW5.1 (A)
- net NEOPIXEL: now reaches U1.25 (IO48)
- net NEOPIXEL: now also R25.1
- net BTN_UP: now reaches U1.26 (IO45)
- net BTN_UP: now also C28.1, R26.2, SW4.1 (A)
- net GPIO35: now reaches U1.28 (IO35)
- net GPIO35: now also J10.3 (Pin_3)
- net GPIO36: now reaches U1.29 (IO36)
- net GPIO36: now also J10.4 (Pin_4)
- net GPIO37: now reaches U1.30 (IO37)
- net GPIO37: now also J10.5 (Pin_5)
- net GPIO38: now reaches U1.31 (IO38)
- net GPIO38: now also J10.6 (Pin_6)
- net BTN_BACK: now reaches U1.38 (IO2)
- net BTN_BACK: now also C31.1, R29.2, SW7.1 (A)
- net GLITCH_ARM: now reaches U1.6 (IO6)
- net GLITCH_ARM: now also SW1.1 (B), LED2.2, R32.2
- net LED_STATUS: now reaches U1.7 (IO7)
- net LED_STATUS: now also R30.2
- net SPI_CS_SD: now reaches U1.8 (IO15)
- net SPI_CS_SD: now also J7.2 (DAT3/CD), R16.1
- net SD_DETECT: now reaches U1.9 (IO16)
- net SD_DETECT: now also J7.9 (DET_LEVER)
- removed net GLITCH_GATE_SW: R17.1, SW1.1 (B)
- new net: LED4.4 (DIN), R25.2
- new net: LED8.2 (DOUT), LED9.4 (DIN)
- new net: D3.1, R30.1
- new net: D4.1, R5.2
- new net: LED2.1, R19.1
- new net: LED6.2 (DOUT), LED7.4 (DIN)
- new net: LED5.2 (DOUT), LED6.4 (DIN)
- new net: LED4.2 (DOUT), LED5.4 (DIN)
- new net: LED7.2 (DOUT), LED8.4 (DIN)
- new net FLASH_VCC: C15.1, SJ1.1 (A), U6.8 (VCC)
- new net SHIELD2: C888.1, J2.S1 (SHIELD), R888.1
- no-connect marks 12 -> 16
Other:
- note added: "10ms RC"
- note added: "Note cathode in symbol edit (this is weird as it seems reversed based on image)!!"
- moved on the sheet: BZ1, C1, C13, C14, C15, C16, C17, C2, C3, C4, C5, C6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
